File: micro-midi.sch (KiCad schematic (older format))
At the start: 15 parts, among them J1 AudioJack3, J2 Conn_01x04_Male, J3 AudioJack3, U1 74HC04, U2 6N137, U3 74AHC04

Commit message: found the right footprint for the 6n137
Parts:
- U2: footprint Package_DIP:DIP-8_W7.62mm -> Package_DIP:PowerIntegrations_SMD-8
Changed lines of the file:
@@
 F 0 "U2" H 5000 3267 50  0000 C CNN
 F 1 "6N137" H 5000 3176 50  0000 C CNN
-F 2 "Package_DIP:DIP-8_W7.62mm" H 5000 2300 50  0001 C CNN
+F 2 "Package_DIP:PowerIntegrations_SMD-8" H 5000 2300 50  0001 C CNN
 F 3 "https://docs.broadcom.com/docs/AV02-0940EN" H 4150 3350 50  0001 C CNN
 	1    5000 2800

Commit message: update resistor footprints to 0805
Parts:
- R1, R2, R5, R6: footprint Resistor_SMD:R_1206_3216Metric -> Resistor_SMD:R_0805_2012Metric_Pad1.15x1.40mm_HandSolder
- R3, R4: footprint (none) -> Resistor_SMD:R_0805_2012Metric_Pad1.15x1.40mm_HandSolder
Changed lines of the file:
@@
 F 0 "R2" H 5880 2354 50  0000 R CNN
 F 1 "10K" H 5880 2445 50  0000 R CNN
-F 2 "Resistor_SMD:R_1206_3216Metric" V 5880 2400 50  0001 C CNN
+F 2 "Resistor_SMD:R_0805_2012Metric_Pad1.15x1.40mm_HandSolder" V 5880 2400 50  0001 C CNN
 F 3 "~" H 5950 2400 50  0001 C CNN
 	1    5950 2400
@@
 F 0 "R3" V 7743 3450 50  0000 C CNN
 F 1 "470" V 7834 3450 50  0000 C CNN
-F 2 "" V 7880 3450 50  0001 C CNN
+F 2 "Resistor_SMD:R_0805_2012Metric_Pad1.15x1.40mm_HandSolder" V 7880 3450 50  0001 C CNN
 F 3 "~" H 7950 3450 50  0001 C CNN
 	1    7950 3450
@@
 F 0 "R4" V 7743 3950 50  0000 C CNN
 F 1 "470" V 7834 3950 50  0000 C CNN
-F 2 "" V 7880 3950 50  0001 C CNN
+F 2 "Resistor_SMD:R_0805_2012Metric_Pad1.15x1.40mm_HandSolder" V 7880 3950 50  0001 C CNN
 F 3 "~" H 7950 3950 50  0001 C CNN
 	1    7950 3950
@@
 F 0 "R1" V 3943 2800 50  0000 C CNN
 F 1 "220R" V 4034 2800 50  0000 C CNN
-F 2 "Resistor_SMD:R_1206_3216Metric" V 4080 2800 50  0001 C CNN
+F 2 "Resistor_SMD:R_0805_2012Metric_Pad1.15x1.40mm_HandSolder" V 4080 2800 50  0001 C CNN
 F 3 "~" H 4150 2800 50  0001 C CNN
 	1    4150 2800
@@
 F 0 "R5" V 7743 4500 50  0000 C CNN
 F 1 "220R" V 7834 4500 50  0000 C CNN
-F 2 "Resistor_SMD:R_1206_3216Metric" V 7880 4500 50  0001 C CNN
+F 2 "Resistor_SMD:R_0805_2012Metric_Pad1.15x1.40mm_HandSolder" V 7880 4500 50  0001 C CNN
 F 3 "~" H 7950 4500 50  0001 C CNN
 	1    7950 4500
@@
 F 0 "R6" V 7743 5050 50  0000 C CNN
 F 1 "220R" V 7834 5050 50  0000 C CNN
-F 2 "Resistor_SMD:R_1206_3216Metric" V 7880 5050 50  0001 C CNN
+F 2 "Resistor_SMD:R_0805_2012Metric_Pad1.15x1.40mm_HandSolder" V 7880 5050 50  0001 C CNN
 F 3 "~" H 7950 5050 50  0001 C CNN
 	1    7950 5050

Commit message: update all to 0805
Parts:
- D1: footprint Diode_SMD:D_1206_3216Metric -> Diode_SMD:D_0805_2012Metric_Pad1.15x1.40mm_HandSolder
- D2, D3: footprint (none) -> LED_SMD:LED_0805_2012Metric_Pad1.15x1.40mm_HandSolder
Changed lines of the file:
@@
 F 0 "D1" V 4404 3029 50  0000 L CNN
 F 1 "1N4148" V 4495 3029 50  0000 L CNN
-F 2 "Diode_SMD:D_1206_3216Metric" H 4450 2775 50  0001 C CNN
+F 2 "Diode_SMD:D_0805_2012Metric_Pad1.15x1.40mm_HandSolder" H 4450 2775 50  0001 C CNN
 F 3 "https://assets.nexperia.com/documents/data-sheet/1N4148_1N4448.pdf" H 4450 2950 50  0001 C CNN
 	1    4450 2950
@@
 F 0 "D2" H 8443 3195 50  0000 C CNN
 F 1 "LED" H 8443 3286 50  0000 C CNN
-F 2 "" H 8450 3450 50  0001 C CNN
+F 2 "LED_SMD:LED_0805_2012Metric_Pad1.15x1.40mm_HandSolder" H 8450 3450 50  0001 C CNN
 F 3 "~" H 8450 3450 50  0001 C CNN
 	1    8450 3450
@@
 F 0 "D3" H 8443 3695 50  0000 C CNN
 F 1 "LED" H 8443 3786 50  0000 C CNN
-F 2 "" H 8450 3950 50  0001 C CNN
+F 2 "LED_SMD:LED_0805_2012Metric_Pad1.15x1.40mm_HandSolder" H 8450 3950 50  0001 C CNN
 F 3 "~" H 8450 3950 50  0001 C CNN
 	1    8450 3950

Commit message: fix U1A
Parts:
- removed U3: 74AHC04, symbol 74xx:74AHC04
- added unit 1 of U1
Connections:
- net at J2.3 (Pin_3), U1.5: now also U1.1
- net at U1.3: now also U1.2
Changed lines of the file:
@@
-$EndComp
-$Comp
-L 74xx:74AHC04 U3
-U 1 1 5E81332C
-P 6500 4500
-F 0 "U3" H 6500 4817 50  0000 C CNN
-F 1 "74AHC04" H 6500 4726 50  0000 C CNN
-F 2 "" H 6500 4500 50  0001 C CNN
-F 3 "https://assets.nexperia.com/documents/data-sheet/74AHC_AHCT04.pdf" H 6500 4500 50  0001 C CNN
-	1    6500 4500
-	1    0    0    -1
 $EndComp
 $Comp
@@
 Wire Wire Line
 	8250 5150 8250 5350
+$Comp
+L 74xx:74HC04 U1
+U 1 1 5EA9FAAC
+P 6500 4500
+F 0 "U1" H 6500 4817 50  0000 C CNN
+F 1 "74HC04" H 6500 4726 50  0000 C CNN
+F 2 "Package_SO:SOIC-14_3.9x8.7mm_P1.27mm" H 6500 4500 50  0001 C CNN
+F 3 "https://assets.nexperia.com/documents/data-sheet/74HC_HCT04.pdf" H 6500 4500 50  0001 C CNN
+	1    6500 4500
+	1    0    0    -1
+$EndComp
 $EndSCHEMATC

Commit message: add pinheader footprint
Parts:
- J2: footprint (none) -> Connector_PinHeader_2.54mm:PinHeader_1x04_P2.54mm_Vertical
Changed lines of the file:
@@
 F 0 "J2" H 7300 3050 50  0000 R CNN
 F 1 "Conn_01x04_Male" H 7150 3050 50  0000 R CNN
-F 2 "" H 7200 2800 50  0001 C CNN
+F 2 "Connector_PinHeader_2.54mm:PinHeader_1x04_P2.54mm_Vertical" H 7200 2800 50  0001 C CNN
 F 3 "~" H 7200 2800 50  0001 C CNN
 	1    7200 2800
